File: BluePill.brd (EAGLE design)
At the start: 23 x 53 mm, 67 parts, among them Q1 32.768kHz, Q2 8MHz, U1 STM32F103C8T6, U2 AMS1117-3.3

Commit message: Fix some warnings
Parts:
- renumbered JP5 to BOOT0, JP6 to BOOT1
Connections:
- net +3V3: now also U2.4
Routing:
- net GND: track 209.1 -> 204.3 mm
- net +3V3: track 135.2 -> 138.9 mm
- added copper zone on layer 1, net +3V3
- removed copper zone on layer 1, net HEAT
Other:
- board text added: "BOOT0"
- board text added: "BOOT1"
- board text added: "C13 OUT"
- board text added: "C14 OUT"
- board text added: "C15 OUT"
