File: BluePill.sch (EAGLE design)
At the start: 67 parts, among them Q1 32.768kHz, Q2 8MHz, U1 STM32F103C8T6, U2 AMS1117-3.3

Commit message: Fix some warnings
Parts:
- renumbered JP5 to BOOT0, JP6 to BOOT1
Other:
- moved on the sheet: U2
Changed lines of the file:
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@@
 <attribute name="LCSC" value="C25741"/>
 </part>
-<part name="JP5" library="SparkFun-Jumpers" deviceset="JUMPER-SMT_3_1-NC_TRACE" device="_NO-SILK" package3d_urn="urn:adsk.eagle:package:39287/1"/>
-<part name="JP6" library="SparkFun-Jumpers" deviceset="JUMPER-SMT_3_1-NC_TRACE" device="_NO-SILK" package3d_urn="urn:adsk.eagle:package:39287/1"/>
+<part name="BOOT0" library="SparkFun-Jumpers" deviceset="JUMPER-SMT_3_1-NC_TRACE" device="_NO-SILK" package3d_urn="urn:adsk.eagle:package:39287/1"/>
+<part name="BOOT1" library="SparkFun-Jumpers" deviceset="JUMPER-SMT_3_1-NC_TRACE" device="_NO-SILK" package3d_urn="urn:adsk.eagle:package:39287/1"/>
 <part name="U$1" library="tactile" deviceset="TACTILE-SWITCH" device="">
 <attribute name="LCSC" value="C318884"/>
@@
 <attribute name="LCSC" x="215.9" y="76.2" size="1.778" layer="96" rot="R270" display="off"/>
 </instance>
-<instance part="JP5" gate="G$1" x="177.8" y="88.9" smashed="yes" rot="R90">
+<instance part="BOOT0" gate="G$1" x="177.8" y="88.9" smashed="yes" rot="R90">
 <attribute name="NAME" x="177.419" y="91.44" size="1.778" layer="95" font="vector" rot="R90"/>
 </instance>
-<instance part="JP6" gate="G$1" x="215.9" y="88.9" smashed="yes" rot="R90">
+<instance part="BOOT1" gate="G$1" x="215.9" y="88.9" smashed="yes" rot="R90">
 <attribute name="NAME" x="215.519" y="91.44" size="1.778" layer="95" font="vector" rot="R90"/>
 </instance>
@@
 </segment>
 <segment>
-<pinref part="JP5" gate="G$1" pin="3"/>
+<pinref part="BOOT0" gate="G$1" pin="3"/>
 <wire x1="182.88" y1="88.9" x2="185.42" y2="88.9" width="0.1524" layer="91"/>
 <pinref part="GND2" gate="1" pin="GND"/>
 </segment>
 <segment>
-<pinref part="JP6" gate="G$1" pin="3"/>
+<pinref part="BOOT1" gate="G$1" pin="3"/>
 <wire x1="220.98" y1="88.9" x2="223.52" y2="88.9" width="0.1524" layer="91"/>
 <pinref part="GND1" gate="1" pin="GND"/>
@@
 <segment>
 <pinref part="R33" gate="G$1" pin="2"/>
-<pinref part="JP5" gate="G$1" pin="2"/>
+<pinref part="BOOT0" gate="G$1" pin="2"/>
 <wire x1="177.8" y1="81.28" x2="177.8" y2="83.82" width="0.1524" layer="91"/>
 </segment>
@@
 <net name="N$2" class="0">
 <segment>
-<pinref part="JP6" gate="G$1" pin="2"/>
+<pinref part="BOOT1" gate="G$1" pin="2"/>
 <pinref part="R34" gate="G$1" pin="1"/>
 <wire x1="215.9" y1="83.82" x2="215.9" y2="81.28" width="0.1524" layer="91"/>
@@
 <net name="+3V3" class="0">
 <segment>
-<pinref part="JP5" gate="G$1" pin="1"/>
+<pinref part="BOOT0" gate="G$1" pin="1"/>
 <wire x1="172.72" y1="88.9" x2="170.18" y2="88.9" width="0.1524" layer="91"/>
 <pinref part="+3V1" gate="G$1" pin="+3V3"/>
@@
 </segment>
 <segment>
-<pinref part="JP6" gate="G$1" pin="1"/>
+<pinref part="BOOT1" gate="G$1" pin="1"/>
 <wire x1="210.82" y1="88.9" x2="208.28" y2="88.9" width="0.1524" layer="91"/>
 <pinref part="+3V3" gate="G$1" pin="+3V3"/>
